Commit message: add src

File: src/h3_simulation/urdf/lidar_front.xacro (robot description, xacro)
@@ -24,13 +24,13 @@
     <gazebo reference="laser_frame_front">
         <material>Gazebo/Red</material>
-        <sensor name="laser" type="ray">
+        <sensor name="laser_front" type="ray">
             <pose> 0 0 0 0 0 0 </pose>
             <visualize>true</visualize>
-            <update_rate>10</update_rate>
+            <update_rate>20</update_rate>
             <ray>
                 <scan>
                     <horizontal>
-                        <samples>360</samples>
-                        <resolution>0.35</resolution>
+                        <samples>1080</samples> <!--Tăng số tia quét-->
+                        <resolution>1</resolution> <!--Tránh nội suy lệch-->
                         <min_angle>-1.6</min_angle>
                         <max_angle>3.1</max_angle>
@@ -42,7 +42,7 @@
                 </range>
             </ray>
-            <plugin name="laser_controller" filename="libgazebo_ros_ray_sensor.so">
+            <plugin name="laser_front_controller" filename="libgazebo_ros_ray_sensor.so">
                 <ros>
-                    <argument>~/out:=scan</argument>
+                    <argument>~/out:=scan_front</argument>
                 </ros>
                 <output_type>sensor_msgs/LaserScan</output_type>

File: src/h3_simulation/urdf/lidar_rear.xacro (robot description, xacro)
@@ -24,25 +24,25 @@
     <gazebo reference="laser_frame_rear">
         <material>Gazebo/Red</material>
-        <sensor name="laser" type="ray">
+        <sensor name="laser_rear" type="ray">
             <pose> 0 0 0 0 0 0 </pose>
             <visualize>true</visualize>
-            <update_rate>10</update_rate>
+            <update_rate>20</update_rate>
             <ray>
                 <scan>
                     <horizontal>
-                        <samples>360</samples>
+                        <samples>1080</samples>
                         <resolution>1</resolution>
-                        <min_angle>-3.14</min_angle>
-                        <max_angle>3.14</max_angle>
+                        <min_angle>-4.7</min_angle>
+                        <max_angle>0.0</max_angle>
                     </horizontal>
                 </scan>
                 <range>
-                    <min>0.3</min>
-                    <max>12</max>
+                    <min>0.05</min>
+                    <max>25</max>
                 </range>
             </ray>
-            <plugin name="laser_controller" filename="libgazebo_ros_ray_sensor.so">
+            <plugin name="laser_rear_controller" filename="libgazebo_ros_ray_sensor.so">
                 <ros>
-                    <argument>~/out:=scan</argument>
+                    <argument>~/out:=scan_rear</argument>
                 </ros>
                 <output_type>sensor_msgs/LaserScan</output_type>

File: src/h3_simulation/urdf/robot.urdf.xacro (robot description, xacro)
@@ -3,5 +3,5 @@
     <xacro:include filename="robot_core.xacro" />
     <xacro:include filename="lidar_front.xacro" />
-    <!-- <xacro:include filename="lidar_rear.xacro" /> -->
+    <xacro:include filename="lidar_rear.xacro" />
     <xacro:include filename="gazebo_control.xacro" />
 </robot>

File: src/h3_simulation/urdf/robot_core.xacro (robot description, xacro)
@@ -216,6 +216,28 @@
         </xacro:inertial_box>
     </link>
-    <gazebo reference="cargo">
-        <material>Gazebo/Orange</material>
-    </gazebo>
+    <!-- Laser Frame -->
+    <!-- <joint name="laser_frame" type="fixed">
+        <parent link="base_link"/>
+        <child link="laser_frame"/>
+        <origin xyz="0 0 0.2" rpy="0 0 0"/>
+    </joint>
+    <link name="laser_frame">
+        <visual>
+            <geometry>
+                <box size="0.1 0.1 0.1"/>
+            </geometry>
+            <material name="red"/>
+        </visual>
+        <collision>
+            <geometry>
+                <box size="0.1 0.1 0.1"/>
+            </geometry>
+        </collision>
+        <xacro:inertial_box mass="0.1" x="0.1" y="0.1" z="0.1">
+            <origin xyz="0 0 0" rpy="0 0 0"/>
+        </xacro:inertial_box>
+    </link>
+    <gazebo reference="laser_frame">
+        <material>Gazebo/Red</material>
+    </gazebo> -->
 </robot>
