Commit message: add docker

File: src/robot_simulation/urdf/lidar.xacro (robot description, xacro)
@@ -4,5 +4,5 @@
         <parent link="base_link"/>
         <child link="laser_frame_front"/>
-        <origin xyz="-0.1 0 0.175" rpy="0 0 0"/>
+        <origin xyz="0.18 0.13 0.065" rpy="0 0 0"/>
     </joint>
     <link name="laser_frame_front">
@@ -33,5 +33,5 @@
                         <samples>1080</samples> <!--Tăng số tia quét-->
                         <resolution>1</resolution> <!--Tránh nội suy lệch-->
-                        <min_angle>-3.14</min_angle>
+                        <min_angle>-1.57</min_angle>
                         <max_angle>3.14</max_angle>
                     </horizontal>

File: src/robot_simulation/urdf/robot_core.xacro (robot description, xacro)
@@ -2,18 +2,17 @@
 <robot xmlns:xacro="http://www.ros.org/wiki/xacro" >
     <xacro:include filename="inertial_macros.xacro"/>
-    <xacro:property name="chassis_length" value="0.335"/>
-    <xacro:property name="chassis_width" value="0.265"/>
-    <xacro:property name="chassis_height" value="0.138"/>
+    <xacro:property name="chassis_length" value="0.4"/>
+    <xacro:property name="chassis_width" value="0.3"/>
+    <xacro:property name="chassis_height" value="0.1"/>
     <xacro:property name="chassis_mass" value="1.0"/>
     <xacro:property name="wheel_radius" value="0.033"/>
     <xacro:property name="wheel_thickness" value="0.026"/>
     <xacro:property name="wheel_mass" value="0.05"/>
-    <xacro:property name="wheel_offset_x" value="0.226"/>
-    <xacro:property name="wheel_offset_y" value="0.1485"/>
-    <xacro:property name="wheel_offset_z" value="0.01"/>
+    <xacro:property name="wheel_offset_x" value="0.15"/>
+    <xacro:property name="wheel_offset_y" value="0.163"/>
+    <xacro:property name="wheel_offset_z" value="0.05"/>
     <xacro:property name="caster_wheel_radius" value="0.01"/>
     <xacro:property name="caster_wheel_mass" value="2"/>
-    <xacro:property name="caster_wheel_offset_x" value="0.075"/>
-    <xacro:property name="caster_wheel_offset_z" value="${wheel_offset_z - wheel_radius + caster_wheel_radius}"/>
+    <xacro:property name="caster_wheel_offset_z" value="0.02295"/>
     <material name="white">
         <color rgba="1 1 1 1" />
@@ -34,13 +33,12 @@
     <link name="base_link">
     </link>
-    <!-- CHASSIS LINK -->
-    <joint name="chassis_joint" type="fixed">
+    <!-- CHASSIS -->
+    <joint name="base_to_chassis" type="fixed">
         <parent link="base_link"/>
         <child link="chassis"/>
-        <origin xyz="${-wheel_offset_x} 0 ${-wheel_offset_z}"/>
+        <origin xyz="0 0 0" rpy="0 0 0"/>
     </joint>
     <link name="chassis">
         <visual>
-            <origin xyz="${chassis_length/2} 0 ${chassis_height/2}"/>
             <geometry>
                 <box size="${chassis_length} ${chassis_width} ${chassis_height}"/>
@@ -49,11 +47,10 @@
         </visual>
         <collision>
-            <origin xyz="${chassis_length/2} 0 ${chassis_height/2}"/>
             <geometry>
                 <box size="${chassis_length} ${chassis_width} ${chassis_height}"/>
             </geometry>
         </collision>
-        <xacro:inertial_box mass="0.5" x="${chassis_length}" y="${chassis_width}" z="${chassis_height}">
-            <origin xyz="${chassis_length/2} 0 ${chassis_height/2}" rpy="0 0 0"/>
+        <xacro:inertial_box mass="${chassis_mass}" x="${chassis_length}" y="${chassis_width}" z="${chassis_height}">
+            <origin xyz="0 0 0" rpy="0 0 0"/>
         </xacro:inertial_box>
     </link>
@@ -61,9 +58,9 @@
         <material>Gazebo/Orange</material>
     </gazebo>
-    <!-- LEFT WHEEL LINK -->
+    <!-- LEFT WHEEL -->
     <joint name="left_wheel_joint" type="continuous">
         <parent link="base_link"/>
         <child link="left_wheel"/>
-        <origin xyz="0 ${wheel_offset_y} 0" rpy="-${pi/2} 0 0" />
+        <origin xyz="0 ${wheel_offset_y} ${-wheel_offset_z}" rpy="-${pi/2} 0 0" />
         <axis xyz="0 0 1"/>
     </joint>
@@ -87,9 +84,9 @@
         <material>Gazebo/Blue</material>
     </gazebo>
-    <!-- RIGHT WHEEL LINK -->
+    <!-- RIGHT WHEEL -->
     <joint name="right_wheel_joint" type="continuous">
         <parent link="base_link"/>
         <child link="right_wheel"/>
-        <origin xyz="0 ${-wheel_offset_y} 0" rpy="${pi/2} 0 0" />
+        <origin xyz="0 ${-wheel_offset_y} ${-wheel_offset_z}" rpy="${pi/2} 0 0" />
         <axis xyz="0 0 -1"/>
     </joint>
@@ -113,11 +110,36 @@
         <material>Gazebo/Blue</material>
     </gazebo>
-    <!-- CASTER WHEEL LINK -->
-    <joint name="caster_wheel_joint" type="fixed">
-        <parent link="chassis"/>
-        <child link="caster_wheel"/>
-        <origin xyz="${caster_wheel_offset_x} 0 ${caster_wheel_offset_z}"/>
-    </joint>
-    <link name="caster_wheel">
+    <!-- CONNECT CHASSIS TO CASTER WHEEL FRONT -->
+    <joint name="connect_caster_wheel_front_joint" type="fixed">
+        <parent link="base_link"/>
+        <child link="connect_caster_wheel_front"/>
+        <origin xyz="${wheel_offset_x} 0 ${-wheel_offset_z}" rpy="0 0 0" />
+    </joint>
+    <link name="connect_caster_wheel_front">
+        <visual>
+            <geometry>
+                <cylinder radius="0.02" length="0.052"/>
+            </geometry>
+            <material name="black"/>
+        </visual>
+        <collision>
+            <geometry>
+                <cylinder radius="0.02" length="0.052"/>
+            </geometry>
+        </collision>
+        <xacro:inertial_cylinder mass="0" length="0.052" radius="0.02">
+            <origin xyz="0 0 0" rpy="0 0 0"/>
+        </xacro:inertial_cylinder>
+    </link>
+    <gazebo reference="connect_caster_wheel_front">
+        <material>Gazebo/Black</material>
+    </gazebo>
+    <!-- CASTER WHEEL FRONT -->
+    <joint name="caster_wheel_front_joint" type="fixed">
+        <parent link="connect_caster_wheel_front"/>
+        <child link="caster_wheel_front"/>
+        <origin xyz="0 0 ${-caster_wheel_offset_z}" rpy="0 0 0" />
+    </joint>
+    <link name="caster_wheel_front">
         <visual>
             <geometry>
@@ -135,8 +157,111 @@
         </xacro:inertial_sphere>
     </link>
-    <gazebo reference="caster_wheel">
+    <gazebo reference="caster_wheel_front">
         <material>Gazebo/White</material>
         <mu1 value="0.001"/>
         <mu2 value="0.001"/>
     </gazebo>
+    <!-- CONNECT CHASSIS TO CASTER WHEEL REAR -->
+    <joint name="connect_caster_wheel_rear_joint" type="fixed">
+        <parent link="base_link"/>
+        <child link="connect_caster_wheel_rear"/>
+        <origin xyz="${-wheel_offset_x} 0 ${-wheel_offset_z}" rpy="0 0 0" />
+    </joint>
+    <link name="connect_caster_wheel_rear">
+        <visual>
+            <geometry>
+                <cylinder radius="0.02" length="0.052"/>
+            </geometry>
+            <material name="black"/>
+        </visual>
+        <collision>
+            <geometry>
+                <cylinder radius="0.02" length="0.052"/>
+            </geometry>
+        </collision>
+        <xacro:inertial_cylinder mass="0" length="0.052" radius="0.02">
+            <origin xyz="0 0 0" rpy="0 0 0"/>
+        </xacro:inertial_cylinder>
+    </link>
+    <gazebo reference="connect_caster_wheel_rear">
+        <material>Gazebo/Black</material>
+    </gazebo>
+    <!-- CASTER WHEEL REAR -->
+    <joint name="caster_wheel_rear_joint" type="fixed">
+        <parent link="connect_caster_wheel_rear"/>
+        <child link="caster_wheel_rear"/>
+        <origin xyz="0 0 ${-caster_wheel_offset_z}" rpy="0 0 0" />
+    </joint>
+    <link name="caster_wheel_rear">
+        <visual>
+            <geometry>
+                <sphere radius="${caster_wheel_radius}"/>
+            </geometry>
+            <material name="white"/>
+        </visual>
+        <collision>
+            <geometry>
+                <sphere radius="${caster_wheel_radius}"/>
+            </geometry>
+        </collision>
+        <xacro:inertial_sphere mass="${caster_wheel_mass}" radius="${caster_wheel_radius}">
+            <origin xyz="0 0 0" rpy="0 0 0"/>
+        </xacro:inertial_sphere>
+    </link>
+    <gazebo reference="caster_wheel_rear">
+        <material>Gazebo/White</material>
+        <mu1 value="0.001"/>
+        <mu2 value="0.001"/>
+    </gazebo>
+    <!-- Connect chassis to cargo -->
+    <joint name="chassis_to_cargo_joint" type="fixed">
+        <parent link="base_link"/>
+        <child link="connect_cargo"/>
+        <origin xyz="0 0 0.065"/>
+    </joint>
+    <link name="connect_cargo">
+        <visual>
+            <origin xyz="0 0 0"/>
+            <geometry>
+                <box size="0.3 0.2 0.03"/>
+            </geometry>
+            <material name="blue"/>
+        </visual>
+        <collision>
+            <origin xyz="0 0 0"/>
+            <geometry>
+                <box size="0.3 0.2 0.03"/>
+            </geometry>
+        </collision>
+        <xacro:inertial_box mass="0.1" x="0.3" y="0.2" z="0.03">
+            <origin xyz="0 0 0" rpy="0 0 0"/>
+        </xacro:inertial_box>
+    </link>
+    <!-- CARGO -->
+    <joint name="cargo_joint" type="fixed">
+        <parent link="connect_cargo"/>
+        <child link="cargo"/>
+        <origin xyz="0 0 0.065"/>
+    </joint>
+    <link name="cargo">
+        <visual>
+            <origin xyz="0 0 0"/>
+            <geometry>
+                <box size="0.4 0.3 0.1"/>
+            </geometry>
+            <material name="orange"/>
+        </visual>
+        <collision>
+            <origin xyz="0 0 0"/>
+            <geometry>
+                <box size="0.4 0.3 0.1"/>
+            </geometry>
+        </collision>
+        <xacro:inertial_box mass="0.4" x="0.4" y="0.3" z="0.1">
+            <origin xyz="0 0 0" rpy="0 0 0"/>
+        </xacro:inertial_box>
+    </link>
+    <gazebo reference="cargo">
+        <material>Gazebo/Orange</material>
+    </gazebo>
 </robot>
