Commit message: fix api server

File: src/robot_simulation/urdf/camera.xacro (robot description, xacro)
@@ -3,8 +3,9 @@
     <joint name="camera_joint" type="fixed">
         <parent link="chassis"/>
-        <child link="camera_link"/>
-        <origin xyz="0.276 0 0.181" rpy="0 0 0"/>
+        <child link="camera_frame"/>
+        <!-- xyz: đặt camera ở trung tâm trên nóc robot, rpy: pitch=-pi/2 → nhìn thẳng lên trần -->
+        <origin xyz="0 0 0.18" rpy="0 -1.5707963 0"/>
     </joint>
-    <link name="camera_link">
+    <link name="camera_frame">
         <visual>
             <geometry>
@@ -22,10 +23,10 @@
     </link>
     <joint name="camera_optical_joint" type="fixed">
-        <parent link="camera_link"/>
-        <child link="camera_link_optical"/>
+        <parent link="camera_frame"/>
+        <child link="camera_frame_optical"/>
         <origin xyz="0 0 0" rpy="${-pi/2} 0 ${-pi/2}"/>
     </joint>
-    <link name="camera_link_optical"></link>
-    <gazebo reference="camera_link">
+    <link name="camera_frame_optical"></link>
+    <gazebo reference="camera_frame">
         <material>Gazebo/Black</material>
         <sensor name="camera" type="camera">
@@ -46,5 +47,5 @@
             </camera>
             <plugin name="camera_controller" filename="libgazebo_ros_camera.so">
-                <frame_name>camera_link_optical</frame_name>
+                <frame_name>camera_frame_optical</frame_name>
             </plugin>
         </sensor>
